File: electronica/Etapa de potencia/_autosave-Etapa de potencia.kicad_pcb (KiCad board)
At the start: 2 copper layers, 70 x 45 mm, 25 parts, among them J1 Bornera Resorte, J2 Bornera Resorte, J3 Bornera Resorte, J4 Bornera 4 pines, J5 Header, Q1 MMBT2222, Q2 MMBT2222, Q3 MMBT2222, U1 ATmega328-PU, U2 ULN2003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

Commit message: ending first pcb
Parts:
- removed J2: Bornera Resorte, potenciaFootprints:BorneraKF141R_8Pins
- removed J3: Bornera Resorte, potenciaFootprints:BorneraKF141R_4Pins
- removed J5: Header, Connector_PinHeader_2.54mm:PinHeader_1x04_P2.54mm_Vertical
- removed Q1, Q2, Q3: MMBT2222, Package_TO_SOT_SMD:SOT-23
- removed R3, R4, R5: 1K, Resistor_SMD:R_0805_2012Metric_Pad1.15x1.40mm_HandSolder
- added DHT1: RJ45, Connector_RJ:RJ45_Amphenol_RJHSE5380, F.Cu at (122.6, 130.2)
- added DHT2: RJ45, Connector_RJ:RJ45_Amphenol_RJHSE5380, F.Cu at (143.5, 130.2)
- added HDF & SH1-2: RJ45, Connector_RJ:RJ45_Amphenol_RJHSE5380, F.Cu at (137.8, 57.1)
- added Luces 1-4: RJ45, Connector_RJ:RJ45_Amphenol_RJHSE5380, F.Cu at (93.3, 57.1)
- added SH1: RJ45, Connector_RJ:RJ45_Amphenol_RJHSE5380, F.Cu at (101.3, 130.2)
- added Ven9-10 & Mot1-2: RJ45, Connector_RJ:RJ45_Amphenol_RJHSE5380, F.Cu at (115.6, 57.1)
- added Ventilador 1-4: RJ45, Connector_RJ:RJ45_Amphenol_RJHSE5380, F.Cu at (76.2, 83.2)
- added Ventilador 5-8: RJ45, Connector_RJ:RJ45_Amphenol_RJHSE5380, F.Cu at (76.3, 61.6)
- J1: value Bornera Resorte -> Bornera 4 pines; footprint potenciaFootprints:BorneraKF141R_8Pins -> TerminalBlock:TerminalBlock_Altech_AK300-4_P5.00mm
- U2, U3: moved to F.Cu
- U6: moved to B.Cu
- moved U6 83.6 mm to (113.7, 110.5)
- moved R6 72.4 mm to (148.6, 67.9), turned to 180 degrees
- moved U4 66.5 mm to (121.9, 70.5)
- moved R2 62.8 mm to (116.8, 71.8), turned to 270 degrees
- moved U3 47.8 mm to (92.1, 77.5), turned to 90 degrees
- moved U5 41.7 mm to (131.4, 113.0), turned to 180 degrees
- moved J1 39.8 mm to (74.9, 120.2), turned to 270 degrees
- moved D1 35.9 mm to (142.2, 90.8), turned to 0 degrees
- moved U2 34.4 mm to (88.3, 115.6), turned to 180 degrees
- moved R1 28.5 mm to (98.4, 115.6)
- moved U1 26.1 mm to (102.2, 115.6), turned to 180 degrees
- moved C1 25.5 mm to (92.1, 98.4), turned to 270 degrees
- moved C3 23.7 mm to (105.4, 96.5), turned to 270 degrees
- moved Y1 20.8 mm to (98.4, 94.0), turned to 90 degrees
- moved C2 16.6 mm to (98.4, 100.3)
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Connections:
- J1 pad 1: GND -> +12V
- J1 pad 2: VO1 -> GND
- J1 pad 3: VO2 -> GND
- J1 pad 4: VO3 -> +5V
- U1 pad 11: H1 -> Net-(U1-Pad11)
- U1 pad 27: V2 -> SH_I1
- U1 pad 28: V1 -> SH_I2
- U1 pad 4: Net-(U1-Pad4) -> V2
- U1 pad 5: Net-(U1-Pad5) -> V1
- U2 pad 1: V7 -> V2
- U2 pad 13: VO4 -> VO1
- U2 pad 14: VO3 -> VO2
- U2 pad 15: VO2 -> VO3
- U2 pad 16: VO1 -> VO4
- U2 pad 2: V6 -> V1
- U2 pad 3: V5 -> V3
- U2 pad 5: V3 -> V5
- U2 pad 6: V2 -> V6
- U2 pad 7: V1 -> V7
- U3 pad 1: L4 -> V8
- U3 pad 2: L3 -> V9
- U3 pad 3: L2 -> L1
- U3 pad 4: L1 -> V10
- U3 pad 5: V10 -> L2
- U3 pad 6: V9 -> L3
- U3 pad 7: V8 -> L4
- U5 pad 11: H_I1 -> PSH2
- U5 pad 12: SH2 -> PSH1
- U5 pad 13: SH1 -> M2
- U5 pad 14: M2 -> M1
- U5 pad 15: Tx -> TX
- U5 pad 16: Rx -> RX
- U5 pad 3: M1 -> Joker
- U5 pad 4: H_I2 -> H1
- U6 pad 12: SHO2 -> MO2
- U6 pad 13: SHO2 -> MO1
- U6 pad 14: H01 -> PSHO2
- U6 pad 15: MO2 -> PSHO1
- U6 pad 16: MO1 -> H01
- U6 pad 4: SH1 -> PSH1
- U6 pad 5: SH2 -> PSH2
Routing:
- net GND: track 145.8 -> 456.8 mm, vias 2 -> 6
- net +5V: track 57.5 -> 212.6 mm, vias 2 -> 6
- net PSHO1: track 0.00 -> 60.2 mm
- net PSHO2: track 0.00 -> 57.2 mm
- net VO4: track 10.7 -> 54.5 mm
- net DHT_I2: track 0.00 -> 43.0 mm
- net VO5: track 12.0 -> 54.4 mm
- net DHT_I1: track 0.00 -> 40.9 mm
- net VO6: track 14.0 -> 54.1 mm
- net VO3: track 10.0 -> 49.0 mm
- net DHT_I3: track 0.00 -> 38.1 mm
- net MO1: track 12.4 -> 50.2 mm
- net VO7: track 17.7 -> 52.5 mm
- net M1: track 39.8 -> 5.08 mm, vias 2 -> 0
- net VO2: track 9.49 -> 43.8 mm
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Other:
- board size 70 x 45 mm -> 91.9 x 96.1 mm
- board text added: "+12 GND GND +5"
- board text added: "FUENTE CARGA"
- board text added: "Fitotron V1.0"
- board text removed: "12 5"
- board text removed: "RX TX GND 5V"
